File: hardware/BREAD_Slice.kicad_pcb (KiCad board)
At the start: 2 copper layers, 70 x 100 mm, 21 parts, among them J1 Conn_01x10_Female, J2 Conn_01x08, J3 Conn_01x08, J4 Conn_02x10_Odd_Even, J5 Conn_02x10_Odd_Even, J6 Conn_02x10_Odd_Even, J7 Conn_02x10_Odd_Even

Commit message: review and revise board and update footprints
Parts:
- added J10: Screw_Terminal_01x02, TerminalBlock_TE-Connectivity:TerminalBlock_TE_282834-2_1x02_P2.54mm_Horizontal, F.Cu at (188.5, 118.3)
- added J11: Screw_Terminal_01x02, TerminalBlock_TE-Connectivity:TerminalBlock_TE_282834-2_1x02_P2.54mm_Horizontal, F.Cu at (188.5, 111.3)
- added J12: Screw_Terminal_01x02, TerminalBlock_TE-Connectivity:TerminalBlock_TE_282834-2_1x02_P2.54mm_Horizontal, F.Cu at (188.5, 104.7)
- added J13: Screw_Terminal_01x02, TerminalBlock_TE-Connectivity:TerminalBlock_TE_282834-2_1x02_P2.54mm_Horizontal, F.Cu at (188.5, 98.1)
- added J14: Screw_Terminal_01x02, TerminalBlock_TE-Connectivity:TerminalBlock_TE_282834-2_1x02_P2.54mm_Horizontal, F.Cu at (188.5, 91.5)
- added J15: Screw_Terminal_01x02, TerminalBlock_TE-Connectivity:TerminalBlock_TE_282834-2_1x02_P2.54mm_Horizontal, F.Cu at (188.5, 84.9)
- added J16: Screw_Terminal_01x02, TerminalBlock_TE-Connectivity:TerminalBlock_TE_282834-2_1x02_P2.54mm_Horizontal, F.Cu at (188.5, 78.3)
- added J17: Screw_Terminal_01x02, TerminalBlock_TE-Connectivity:TerminalBlock_TE_282834-2_1x02_P2.54mm_Horizontal, F.Cu at (188.5, 71.3)
- added J4: Screw_Terminal_01x02, TerminalBlock_TE-Connectivity:TerminalBlock_TE_282834-2_1x02_P2.54mm_Horizontal, F.Cu at (172.2, 44.3)
- added J5: Screw_Terminal_01x02, TerminalBlock_TE-Connectivity:TerminalBlock_TE_282834-2_1x02_P2.54mm_Horizontal, F.Cu at (165.6, 44.3)
- added J7: Screw_Terminal_01x02, TerminalBlock_TE-Connectivity:TerminalBlock_TE_282834-2_1x02_P2.54mm_Horizontal, F.Cu at (152.4, 44.3)
- added J8: Screw_Terminal_01x02, TerminalBlock_TE-Connectivity:TerminalBlock_TE_282834-2_1x02_P2.54mm_Horizontal, F.Cu at (145.8, 44.3)
- added J9: Screw_Terminal_01x02, TerminalBlock_TE-Connectivity:TerminalBlock_TE_282834-2_1x02_P2.54mm_Horizontal, F.Cu at (139.2, 44.3)
- A1: footprint Module:Arduino_Nano -> KMLib_Boards_Modules:Arduino_Nano_Headers
- D1: footprint SparkFun-LED:WS2812-5050-4PIN -> KMLib_IC_SMD:WS2812-5050-4PIN
- HS1: footprint KML-Custom:Thermal Pad -> KMLib_Mounting:Thermal Pad
- J2, J3: value Conn_01x08 -> Screw_Terminal_01x02; footprint TerminalBlock_4Ucon:TerminalBlock_4Ucon_1x08_P3.50mm_Horizontal -> TerminalBlock_TE-Connectivity:TerminalBlock_TE_282834-2_1x02_P2.54mm_Horizontal
- J6: value Conn_02x10_Odd_Even -> Screw_Terminal_01x02; footprint Connector_PinHeader_2.54mm:PinHeader_2x10_P2.54mm_Vertical -> TerminalBlock_TE-Connectivity:TerminalBlock_TE_282834-2_1x02_P2.54mm_Horizontal
- moved J3 73.6 mm to (178.8, 44.3), turned to 180 degrees
- moved J2 18.9 mm to (188.5, 64.3)
- moved J6 15.2 mm to (159.0, 44.3), turned to 180 degrees
- moved J20 0.36 mm to (142.6, 59.1)
- renumbered J4 to J18, J5 to J19, J7 to J20
Connections:
- J2 pad 2: /D12 -> GND
- J3 pad 1: /AREF -> /D12
- J3 pad 2: /A0 -> GND
- J6 pad 1: +5V -> /D9
Routing:
- net +5V: track 185.1 -> 152.9 mm
- net /D12: track 82.5 -> 103.9 mm
- net /D11: track 81.8 -> 98.4 mm
- net /D10: track 81.3 -> 93.1 mm
- net /RESET: track 33.2 -> 43.9 mm
- net /D13: track 76.7 -> 85.8 mm
- net /A7: track 33.9 -> 42.8 mm
- net /A6: track 33.5 -> 41.1 mm
- net /D6: track 79.3 -> 86.8 mm
- net /D9: track 80.8 -> 87.9 mm
- net /A3: track 35.2 -> 41.5 mm
- net /D8: track 80.3 -> 86.4 mm
- net /D7: track 79.8 -> 85.7 mm
- net /A2: track 34.8 -> 39.8 mm
- net /A1: track 34.4 -> 38.2 mm
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Other:
- board text added: "GND A0"
- board text added: "GND A1"
- board text added: "GND A2"
- board text added: "GND A3"
- board text added: "GND A6"
- board text added: "GND A7"
- board text added: "GND AREF"
- board text added: "GND D10"
- board text added: "GND D11"
- board text added: "GND D12"
- board text added: "GND D13"
- board text added: "GND D6"
- board text added: "GND D7"
- board text added: "GND D8"
- board text added: "GND D9"
- board text added: "GND RESET"
- board text removed: "A7 A6 A5 A4 A3 A2 A1 A0 AREF"
- board text removed: "D6 D7 D8 D9 D10 D11 D12 D13"
