File: hardware/BREAD_Slice.kicad_sch (KiCad schematic)
At the start: 20 parts, among them J1 Conn_01x10_Female, J2 Conn_01x08, J3 Conn_01x08, J4 Conn_02x10_Odd_Even, J5 Conn_02x10_Odd_Even, J6 Conn_02x10_Odd_Even, J7 Conn_02x10_Odd_Even

Commit message: review and revise board and update footprints
Parts:
- removed J2, J3: Conn_01x08, TerminalBlock_4Ucon:TerminalBlock_4Ucon_1x08_P3.50mm_Horizontal, symbol Connector_Generic:Conn_01x08
- removed J6: Conn_02x10_Odd_Even, Connector_PinHeader_2.54mm:PinHeader_2x10_P2.54mm_Vertical, symbol Connector_Generic:Conn_02x10_Odd_Even
- added J10, J11, J12, J13, J14, J15, J16, J17, J2, J3, J4, J5, J6, J7, J8, J9: Screw_Terminal_01x02, TerminalBlock_TE-Connectivity:TerminalBlock_TE_282834-2_1x02_P2.54mm_Horizontal, symbol Connector:Screw_Terminal_01x02
- A1: footprint Module:Arduino_Nano -> KMLib_Boards_Modules:Arduino_Nano_Headers
- D1: footprint SparkFun-LED:WS2812-5050-4PIN -> KMLib_IC_SMD:WS2812-5050-4PIN
- HS1: footprint KML-Custom:Thermal Pad -> KMLib_Mounting:Thermal Pad
- renumbered J4 to J18, J5 to J19, J7 to J20
Connections:
- net A0: now also J11.1 (Pin_1)
- net A1: now also J12.1 (Pin_1)
- net A2: now also J13.1 (Pin_1)
- net A3: now also J14.1 (Pin_1)
- net A6: now also J15.1 (Pin_1)
- net A7: now also J16.1 (Pin_1)
- net AREF: now also J10.1 (Pin_1)
- net D10: now also J5.1 (Pin_1)
- net D11: now also J4.1 (Pin_1)
- net D12: now also J3.1 (Pin_1)
- net D13: now also J2.1 (Pin_1)
- net D6: now also J9.1 (Pin_1)
- net D7: now also J8.1 (Pin_1)
- net D8: now also J7.1 (Pin_1)
- net D9: now also J6.1 (Pin_1)
- net GND: now also J10.2 (Pin_2), J11.2 (Pin_2), J12.2 (Pin_2), J13.2 (Pin_2), J14.2 (Pin_2), J15.2 (Pin_2), J16.2 (Pin_2), J17.2 (Pin_2), J2.2 (Pin_2), J3.2 (Pin_2), J4.2 (Pin_2), J5.2 (Pin_2), J6.2 (Pin_2), J7.2 (Pin_2), J8.2 (Pin_2), J9.2 (Pin_2)
- net RESET: now also J17.1 (Pin_1)
Other:
- moved on the sheet: J18, J19, J20
